File: N64-PDS.kicad_sch (KiCad schematic)
At the start: 62 parts, among them J1 USB-C-6P-PWR, J2 I2C_OUT, J3 PWR_OUT, U1 STUSB4500QTR, U2 PTPS55289RYQR, U3 STL6P3LLH6, U4 PTPS55289RYQR

Commit message: Finish board layout and routing
Finished board layout and routing, added a hatched ground plane for looks (and some emi)
Parts:
- R5: now not fitted
Connections:
- net at C23.1: now also R17.2; no longer U4.15 (COMP)
- net at C23.2: now also U4.15 (COMP); no longer R17.2
- net at C7.1: now also L1.2, U2.10 (SW2); no longer U2.19 (BOOT2)
- net GND renamed AGND
- new net: C7.2, U2.19 (BOOT2)
Other:
- moved on the sheet: C23, C7, R20
Changed lines of the file:
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@@
 	)
 	(junction
-		(at 207.01 101.6)
-		(diameter 0)
-		(color 0 0 0 0)
-	)
-	(junction
 		(at 194.31 128.27)
 		(diameter 0)
@@
 	)
 	(junction
+		(at 207.01 101.6)
+		(diameter 0)
+		(color 0 0 0 0)
+	)
+	(junction
 		(at 113.03 161.29)
 		(diameter 0)
@@
 	(wire
 		(pts
+			(xy 120.65 190.5) (xy 120.65 193.04)
+		)
+		(stroke
+			(width 0)
+			(type default)
+		)
+	)
+	(wire
+		(pts
 			(xy 44.45 185.42) (xy 46.99 185.42)
 		)
@@
 	)
 	(symbol
+		(lib_id "power:GND")
+		(at 120.65 190.5 180)
+		(unit 1)
+		(exclude_from_sim no)
+		(in_bom yes)
+		(on_board yes)
+		(dnp no)
+		(fields_autoplaced yes)
+		(property "Reference" "#PWR025"
+			(at 120.65 184.15 0)
+			(effects
+				(font
+					(size 1.27 1.27)
+				)
+				(hide yes)
+			)
+		)
+		(property "Value" "AGND"
+			(at 120.65 185.42 0)
+			(effects
+				(font
+					(size 1.27 1.27)
+				)
+				(hide yes)
+			)
+		)
+		(property "Footprint" ""
+			(at 120.65 190.5 0)
+			(effects
+				(font
+					(size 1.27 1.27)
+				)
+				(hide yes)
+			)
+		)
+		(property "Datasheet" ""
+			(at 120.65 190.5 0)
+			(effects
+				(font
+					(size 1.27 1.27)
+				)
+				(hide yes)
+			)
+		)
+		(property "Description" "Power symbol creates a global label with name \"GND\" , ground"
+			(at 120.65 190.5 0)
+			(effects
+				(font
+					(size 1.27 1.27)
+				)
+				(hide yes)
+			)
+		)
+		(pin "1"
+		)
+		(instances
+			(project "N64-PDS"
+				(path "/9649f91c-0b3c-463e-88a6-37fb387993ef"
+					(reference "#PWR025")
+					(unit 1)
+				)
+			)
+		)
+	)
+	(symbol
 		(lib_id "Device:R")
 		(at 34.29 77.47 90)
@@
 	(symbol
 		(lib_id "Device:C")
-		(at 200.66 109.22 270)
+		(at 200.66 109.22 90)
+		(mirror x)
 		(unit 1)
 		(exclude_from_sim no)
@@
 		(dnp no)
 		(property "Reference" "C23"
-			(at 201.676 107.95 90)
+			(at 199.644 107.95 90)
 			(effects
 				(font
@@
 		)
 		(property "Value" "100n"
-			(at 194.564 110.49 90)
+			(at 206.756 110.49 90)
 			(effects
 				(font
@@
 		)
 		(property "Footprint" "Capacitor_SMD:C_0402_1005Metric_Pad0.74x0.62mm_HandSolder"
-			(at 196.85 110.1852 0)
+			(at 204.47 110.1852 0)
 			(effects
 				(font
@@
 	(symbol
 		(lib_id "Device:C")
-		(at 95.25 154.94 90)
+		(at 95.25 154.94 270)
+		(mirror x)
 		(unit 1)
 		(exclude_from_sim no)
@@
 		(dnp no)
 		(property "Reference" "C7"
-			(at 93.726 156.21 90)
+			(at 96.774 156.21 90)
 			(effects
 				(font
@@
 		)
 		(property "Value" "100n"
-			(at 101.346 153.924 90)
+			(at 89.154 153.924 90)
 			(effects
 				(font
@@
 		)
 		(property "Footprint" "Capacitor_SMD:C_0603_1608Metric_Pad1.08x0.95mm_HandSolder"
-			(at 99.06 153.9748 0)
+			(at 91.44 153.9748 0)
 			(effects
 				(font
@@
 		(on_board yes)
 		(dnp no)
-		(fields_autoplaced yes)
 		(property "Reference" "U4"
 			(at 228.6 160.02 0)
@@
 	(symbol
 		(lib_id "Device:R")
-		(at 267.97 143.51 180)
+		(at 267.97 143.51 0)
+		(mirror x)
 		(unit 1)
 		(exclude_from_sim no)
@@
 		(dnp no)
 		(property "Reference" "R20"
-			(at 270.764 139.954 0)
+			(at 265.176 139.954 0)
 			(effects
 				(font
@@
 		)
 		(property "Value" "274"
-			(at 265.684 140.97 90)
+			(at 270.256 140.97 90)
 			(effects
 				(font
@@
 		)
 		(property "Footprint" "Resistor_SMD:R_0402_1005Metric_Pad0.72x0.64mm_HandSolder"
-			(at 269.748 143.51 90)
+			(at 266.192 143.51 90)
 			(effects
 				(font
@@
 	(symbol
 		(lib_id "power:GND")
+		(at 120.65 193.04 0)
+		(mirror y)
+		(unit 1)
+		(exclude_from_sim no)
+		(in_bom yes)
+		(on_board yes)
+		(dnp no)
+		(property "Reference" "#PWR024"
+			(at 120.65 199.39 0)
+			(effects
+				(font
+					(size 1.27 1.27)
+				)
+				(hide yes)
+			)
+		)
+		(property "Value" "GND"
+			(at 120.65 198.12 0)
+			(effects
+				(font
+					(size 1.27 1.27)
+				)
+				(hide yes)
+			)
+		)
+		(property "Footprint" ""
+			(at 120.65 193.04 0)
+			(effects
+				(font
+					(size 1.27 1.27)
+				)
+				(hide yes)
+			)
+		)
+		(property "Datasheet" ""
+			(at 120.65 193.04 0)
+			(effects
+				(font
+					(size 1.27 1.27)
+				)
+				(hide yes)
+			)
+		)
+		(property "Description" "Power symbol creates a global label with name \"GND\" , ground"
+			(at 120.65 193.04 0)
+			(effects
+				(font
+					(size 1.27 1.27)
+				)
+				(hide yes)
+			)
+		)
+		(pin "1"
+		)
+		(instances
+			(project "N64-PDS"
+				(path "/9649f91c-0b3c-463e-88a6-37fb387993ef"
+					(reference "#PWR024")
+					(unit 1)
+				)
+			)
+		)
+	)
+	(symbol
+		(lib_id "power:GND")
 		(at 267.97 101.6 180)
 		(unit 1)
@@
 		(in_bom yes)
 		(on_board yes)
-		(dnp no)
+		(dnp yes)
 		(property "Reference" "R5"
 			(at 32.258 102.87 0)

Commit message: Kicad 9
Connections:
- net I2C_3V3 is gone; now on net VBUS: J2.4 (Pin_4)
- net I2C_SCL: now also J2.3 (Pin_3); no longer J2.2 (Pin_2)
- net I2C_SDA: now also J2.2 (Pin_2); no longer J2.3 (Pin_3)
