File: N64-PDS.kicad_sch (KiCad schematic)
At the start: 62 parts, among them J1 USB-C-6P-PWR, J2 I2C_OUT, J3 PWR_OUT, U1 STUSB4500QTR, U2 PTPS55289RYQR, U3 STL6P3LLH6, U4 PTPS55289RYQR

Commit message: Oops all redesigns
I did it again, this time smaller, better laid out, and all around maybe gooderer
Parts:
- removed C9: 100n, Capacitor_SMD:C_0402_1005Metric_Pad0.74x0.62mm_HandSolder, symbol Device:C
- added C32: 4.7n, Capacitor_SMD:C_0402_1005Metric_Pad0.74x0.62mm_HandSolder, symbol Device:C
- R20: value 274 -> 274k
- R9: value 301 -> 56.2k
Connections:
- net AGND: now also R3.2; no longer R3.1
- net at U1.6 (RESET): now also R3.1; no longer R3.2
- net at U2.15 (COMP): now also C32.2
- net at R9.2: now also C32.1
Other:
- moved on the sheet: R3
Changed lines of the file:
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@@
 	(text "Voltage divider for vcc (5v) to ~3.3v for high"
 		(exclude_from_sim no)
-		(at 48.768 176.784 0)
+		(at 46.736 176.784 0)
 		(effects
 			(font
@@
 	(wire
 		(pts
+			(xy 100.33 180.34) (xy 104.14 180.34)
+		)
+		(stroke
+			(width 0)
+			(type default)
+		)
+	)
+	(wire
+		(pts
 			(xy 176.53 119.38) (xy 166.37 119.38)
 		)
@@
 	(wire
 		(pts
-			(xy 100.33 180.34) (xy 104.14 180.34)
-		)
-		(stroke
-			(width 0)
-			(type default)
-		)
-	)
-	(wire
-		(pts
 			(xy 99.06 154.94) (xy 101.6 154.94)
 		)
@@
 	(symbol
 		(lib_id "Device:R")
-		(at 34.29 77.47 90)
+		(at 34.29 77.47 270)
 		(unit 1)
 		(exclude_from_sim no)
@@
 		(dnp no)
 		(property "Reference" "R3"
-			(at 32.766 79.756 90)
+			(at 35.814 75.184 90)
 			(effects
 				(font
@@
 		)
 		(property "Value" "10k"
-			(at 34.036 75.184 90)
+			(at 34.544 79.756 90)
 			(effects
 				(font
@@
 		)
 		(property "Footprint" "Resistor_SMD:R_0402_1005Metric_Pad0.72x0.64mm_HandSolder"
-			(at 34.29 79.248 90)
+			(at 34.29 75.692 90)
 			(effects
 				(font
@@
 		)
 		(property "Value" "48.7k"
-			(at 256.54 104.14 90)
+			(at 256.286 103.124 90)
 			(effects
 				(font
@@
 	)
 	(symbol
-		(lib_id "Device:C")
-		(at 96.52 180.34 90)
-		(unit 1)
-		(exclude_from_sim no)
-		(in_bom yes)
-		(on_board yes)
-		(dnp no)
-		(property "Reference" "C9"
-			(at 95.504 181.61 90)
-			(effects
-				(font
-					(size 1.27 1.27)
-				)
-				(justify left)
-			)
-		)
-		(property "Value" "100n"
-			(at 102.616 179.07 90)
-			(effects
-				(font
-					(size 1.27 1.27)
-				)
-				(justify left)
-			)
-		)
-		(property "Footprint" "Capacitor_SMD:C_0402_1005Metric_Pad0.74x0.62mm_HandSolder"
-			(at 100.33 179.3748 0)
-			(effects
-				(font
-					(size 1.27 1.27)
-				)
-				(hide yes)
-			)
-		)
-		(property "Datasheet" "~"
-			(at 96.52 180.34 0)
-			(effects
-				(font
-					(size 1.27 1.27)
-				)
-				(hide yes)
-			)
-		)
-		(property "Description" "Unpolarized capacitor"
-			(at 96.52 180.34 0)
-			(effects
-				(font
-					(size 1.27 1.27)
-				)
-				(hide yes)
-			)
-		)
-		(pin "1"
-		)
-		(pin "2"
-		)
-		(instances
-			(project "N64-PDS"
-				(path "/9649f91c-0b3c-463e-88a6-37fb387993ef"
-					(reference "C9")
-					(unit 1)
-				)
-			)
-		)
-	)
-	(symbol
 		(lib_id "power:PWR_FLAG")
 		(at 115.57 78.74 270)
@@
 			)
 		)
-		(property "Value" "301"
+		(property "Value" "56.2k"
 			(at 104.14 182.118 90)
 			(effects
@@
 		)
 		(property "Value" "56.2k"
-			(at 193.04 108.204 90)
+			(at 194.31 107.95 90)
 			(effects
 				(font
@@
 	)
 	(symbol
+		(lib_id "Device:C")
+		(at 96.52 180.34 270)
+		(unit 1)
+		(exclude_from_sim no)
+		(in_bom yes)
+		(on_board yes)
+		(dnp no)
+		(property "Reference" "C32"
+			(at 97.536 179.07 90)
+			(effects
+				(font
+					(size 1.27 1.27)
+				)
+				(justify left)
+			)
+		)
+		(property "Value" "4.7n"
+			(at 90.424 181.61 90)
+			(effects
+				(font
+					(size 1.27 1.27)
+				)
+				(justify left)
+			)
+		)
+		(property "Footprint" "Capacitor_SMD:C_0402_1005Metric_Pad0.74x0.62mm_HandSolder"
+			(at 92.71 181.3052 0)
+			(effects
+				(font
+					(size 1.27 1.27)
+				)
+				(hide yes)
+			)
+		)
+		(property "Datasheet" "~"
+			(at 96.52 180.34 0)
+			(effects
+				(font
+					(size 1.27 1.27)
+				)
+				(hide yes)
+			)
+		)
+		(property "Description" "Unpolarized capacitor"
+			(at 96.52 180.34 0)
+			(effects
+				(font
+					(size 1.27 1.27)
+				)
+				(hide yes)
+			)
+		)
+		(pin "1"
+		)
+		(pin "2"
+		)
+		(instances
+			(project "N64-PDS"
+				(path "/9649f91c-0b3c-463e-88a6-37fb387993ef"
+					(reference "C32")
+					(unit 1)
+				)
+			)
+		)
+	)
+	(symbol
 		(lib_id "STL6P3LLH6:STL6P3LLH6")
 		(at 152.4 53.34 0)
@@
 			)
 		)
-		(property "Value" "274"
+		(property "Value" "274k"
 			(at 267.97 141.478 90)
 			(effects
@@
 		)
 		(property "Value" "48.7k"
-			(at 40.64 185.674 90)
+			(at 40.64 184.15 90)
 			(effects
 				(font
